Commit message: fix: correct dual arm base spacing from 0.3m to 0.415m
Measured physical distance between left and right arm bases is 0.83m,
updated URDF to reflect actual hardware dimensions.

Co-Authored-By: Claude Opus 4.7 (1M context) <noreply@anthropic.com>

File: assets/r5_urdf/dual_R5a.urdf (robot description, URDF)
Before this commit: robot bimanual_R5a, 19 links, 18 joints
Joints:
- joint world_to_left_base: origin xyz=0 0.3 0 rpy=0 0 0 -> xyz=0 0.415 0 rpy=0 0 0
- joint world_to_right_base: origin xyz=0 -0.3 0 rpy=0 0 0 -> xyz=0 -0.415 0 rpy=0 0 0
